File: pcb/solstrejf-modmatrix-pots/solstrejf-modmatrix-pots.kicad_sch (KiCad schematic)
At the start: 8 parts, among them J1 Conn_02x08_Counter_Clockwise, J2 Conn_02x08_Counter_Clockwise, J3 Conn_02x08_Counter_Clockwise, J4 Conn_02x08_Counter_Clockwise

Commit message: updated pcb layout
Connections:
- net V1AMP1: now also J1.15 (Pin_15); no longer J1.16 (Pin_16)
- net V1AMP2: now also J1.13 (Pin_13); no longer J1.11 (Pin_11)
- net V1AMP3: now also J1.12 (Pin_12); no longer J1.10 (Pin_10)
- net V1AMP4: now also J1.6 (Pin_6); no longer J1.4 (Pin_4)
- net V1FREQ1: now also J1.16 (Pin_16); no longer J1.15 (Pin_15)
- net V1FREQ2: now also J1.11 (Pin_11); no longer J1.13 (Pin_13)
- net V1FREQ3: now also J1.10 (Pin_10); no longer J1.12 (Pin_12)
- net V1FREQ4: now also J1.4 (Pin_4); no longer J1.6 (Pin_6)
- net V2AMP1: now also J2.15 (Pin_15); no longer J2.16 (Pin_16)
- net V2AMP2: now also J2.13 (Pin_13); no longer J2.11 (Pin_11)
- net V2AMP3: now also J2.12 (Pin_12); no longer J2.10 (Pin_10)
- net V2AMP4: now also J2.6 (Pin_6); no longer J2.4 (Pin_4)
- net V2FREQ1: now also J2.16 (Pin_16); no longer J2.15 (Pin_15)
- net V2FREQ2: now also J2.11 (Pin_11); no longer J2.13 (Pin_13)
- net V2FREQ3: now also J2.10 (Pin_10); no longer J2.12 (Pin_12)
- net V2FREQ4: now also J2.4 (Pin_4); no longer J2.6 (Pin_6)
- net V3AMP1: now also J3.15 (Pin_15); no longer J3.16 (Pin_16)
- net V3AMP2: now also J3.13 (Pin_13); no longer J3.11 (Pin_11)
- net V3AMP3: now also J3.12 (Pin_12); no longer J3.10 (Pin_10)
- net V3AMP4: now also J3.6 (Pin_6); no longer J3.4 (Pin_4)
- net V3FREQ1: now also J3.16 (Pin_16); no longer J3.15 (Pin_15)
- net V3FREQ2: now also J3.11 (Pin_11); no longer J3.13 (Pin_13)
- net V3FREQ3: now also J3.10 (Pin_10); no longer J3.12 (Pin_12)
- net V3FREQ4: now also J3.4 (Pin_4); no longer J3.6 (Pin_6)
- net V4AMP1: now also J4.15 (Pin_15); no longer J4.16 (Pin_16)
- net V4AMP2: now also J4.13 (Pin_13); no longer J4.11 (Pin_11)
- net V4AMP3: now also J4.12 (Pin_12); no longer J4.10 (Pin_10)
- net V4AMP4: now also J4.6 (Pin_6); no longer J4.4 (Pin_4)
- net V4FREQ1: now also J4.16 (Pin_16); no longer J4.15 (Pin_15)
- net V4FREQ2: now also J4.11 (Pin_11); no longer J4.13 (Pin_13)
- net V4FREQ3: now also J4.10 (Pin_10); no longer J4.12 (Pin_12)
- net V4FREQ4: now also J4.4 (Pin_4); no longer J4.6 (Pin_6)
Changed lines of the file:
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@@
 	)
 	(label "V4FREQ4"
-		(at 270.51 125.73 0)
+		(at 270.51 123.19 0)
 		(fields_autoplaced yes)
 		(effects
@@
 	)
 	(label "V4AMP3"
-		(at 270.51 130.81 0)
+		(at 270.51 133.35 0)
 		(fields_autoplaced yes)
 		(effects
@@
 	)
 	(label "V2FREQ3"
-		(at 270.51 69.85 0)
+		(at 270.51 67.31 0)
 		(fields_autoplaced yes)
 		(effects
@@
 	)
 	(label "V2AMP4"
-		(at 270.51 59.69 0)
+		(at 270.51 62.23 0)
 		(fields_autoplaced yes)
 		(effects
@@
 	)
 	(label "V3FREQ4"
-		(at 137.16 125.73 0)
+		(at 137.16 123.19 0)
 		(fields_autoplaced yes)
 		(effects
@@
 	)
 	(label "V2FREQ2"
-		(at 257.81 72.39 180)
+		(at 257.81 69.85 180)
 		(fields_autoplaced yes)
 		(effects
@@
 	)
 	(label "V1AMP3"
-		(at 137.16 67.31 0)
+		(at 137.16 69.85 0)
 		(fields_autoplaced yes)
 		(effects
@@
 	)
 	(label "V1FREQ3"
-		(at 137.16 69.85 0)
+		(at 137.16 67.31 0)
 		(fields_autoplaced yes)
 		(effects
@@
 	)
 	(label "V2FREQ4"
-		(at 270.51 62.23 0)
+		(at 270.51 59.69 0)
 		(fields_autoplaced yes)
 		(effects
@@
 	)
 	(label "V1AMP2"
-		(at 124.46 69.85 180)
+		(at 124.46 72.39 180)
 		(fields_autoplaced yes)
 		(effects
@@
 	)
 	(label "V4FREQ3"
-		(at 270.51 133.35 0)
+		(at 270.51 130.81 0)
 		(fields_autoplaced yes)
 		(effects
@@
 	)
 	(label "V2AMP3"
-		(at 270.51 67.31 0)
+		(at 270.51 69.85 0)
 		(fields_autoplaced yes)
 		(effects
@@
 	)
 	(label "V1AMP1"
-		(at 137.16 74.93 0)
-		(fields_autoplaced yes)
-		(effects
-			(font
-				(size 1.27 1.27)
-			)
-			(justify left bottom)
+		(at 124.46 74.93 180)
+		(fields_autoplaced yes)
+		(effects
+			(font
+				(size 1.27 1.27)
+			)
+			(justify right bottom)
 		)
 	)
@@
 	)
 	(label "V4AMP2"
-		(at 257.81 133.35 180)
+		(at 257.81 135.89 180)
 		(fields_autoplaced yes)
 		(effects
@@
 	)
 	(label "V3AMP4"
-		(at 137.16 123.19 0)
+		(at 137.16 125.73 0)
 		(fields_autoplaced yes)
 		(effects
@@
 	)
 	(label "V3FREQ3"
-		(at 137.16 133.35 0)
+		(at 137.16 130.81 0)
 		(fields_autoplaced yes)
 		(effects
@@
 	)
 	(label "V3FREQ2"
-		(at 124.46 135.89 180)
+		(at 124.46 133.35 180)
 		(fields_autoplaced yes)
 		(effects
@@
 	)
 	(label "V2FREQ1"
-		(at 257.81 74.93 180)
-		(fields_autoplaced yes)
-		(effects
-			(font
-				(size 1.27 1.27)
-			)
-			(justify right bottom)
+		(at 270.51 74.93 0)
+		(fields_autoplaced yes)
+		(effects
+			(font
+				(size 1.27 1.27)
+			)
+			(justify left bottom)
 		)
 	)
@@
 	)
 	(label "V4AMP4"
-		(at 270.51 123.19 0)
+		(at 270.51 125.73 0)
 		(fields_autoplaced yes)
 		(effects
@@
 	)
 	(label "V3FREQ1"
-		(at 124.46 138.43 180)
-		(fields_autoplaced yes)
-		(effects
-			(font
-				(size 1.27 1.27)
-			)
-			(justify right bottom)
+		(at 137.16 138.43 0)
+		(fields_autoplaced yes)
+		(effects
+			(font
+				(size 1.27 1.27)
+			)
+			(justify left bottom)
 		)
 	)
@@
 	)
 	(label "V1FREQ1"
-		(at 124.46 74.93 180)
-		(fields_autoplaced yes)
-		(effects
-			(font
-				(size 1.27 1.27)
-			)
-			(justify right bottom)
+		(at 137.16 74.93 0)
+		(fields_autoplaced yes)
+		(effects
+			(font
+				(size 1.27 1.27)
+			)
+			(justify left bottom)
 		)
 	)
 	(label "V3AMP2"
-		(at 124.46 133.35 180)
+		(at 124.46 135.89 180)
 		(fields_autoplaced yes)
 		(effects
@@
 	)
 	(label "V2AMP1"
-		(at 270.51 74.93 0)
-		(fields_autoplaced yes)
-		(effects
-			(font
-				(size 1.27 1.27)
-			)
-			(justify left bottom)
+		(at 257.81 74.93 180)
+		(fields_autoplaced yes)
+		(effects
+			(font
+				(size 1.27 1.27)
+			)
+			(justify right bottom)
 		)
 	)
 	(label "V1FREQ4"
-		(at 137.16 62.23 0)
+		(at 137.16 59.69 0)
 		(fields_autoplaced yes)
 		(effects
@@
 	)
 	(label "V2AMP2"
-		(at 257.81 69.85 180)
+		(at 257.81 72.39 180)
 		(fields_autoplaced yes)
 		(effects
@@
 	)
 	(label "V3AMP1"
-		(at 137.16 138.43 0)
-		(fields_autoplaced yes)
-		(effects
-			(font
-				(size 1.27 1.27)
-			)
-			(justify left bottom)
+		(at 124.46 138.43 180)
+		(fields_autoplaced yes)
+		(effects
+			(font
+				(size 1.27 1.27)
+			)
+			(justify right bottom)
 		)
 	)
@@
 	)
 	(label "V4AMP1"
-		(at 270.51 138.43 0)
-		(fields_autoplaced yes)
-		(effects
-			(font
-				(size 1.27 1.27)
-			)
-			(justify left bottom)
+		(at 257.81 138.43 180)
+		(fields_autoplaced yes)
+		(effects
+			(font
+				(size 1.27 1.27)
+			)
+			(justify right bottom)
 		)
 	)
@@
 	)
 	(label "V4FREQ1"
-		(at 257.81 138.43 180)
-		(fields_autoplaced yes)
-		(effects
-			(font
-				(size 1.27 1.27)
-			)
-			(justify right bottom)
+		(at 270.51 138.43 0)
+		(fields_autoplaced yes)
+		(effects
+			(font
+				(size 1.27 1.27)
+			)
+			(justify left bottom)
 		)
 	)
@@
 	)
 	(label "V3AMP3"
-		(at 137.16 130.81 0)
+		(at 137.16 133.35 0)
 		(fields_autoplaced yes)
 		(effects
@@
 	)
 	(label "V1AMP4"
-		(at 137.16 59.69 0)
+		(at 137.16 62.23 0)
 		(fields_autoplaced yes)
 		(effects
@@
 	)
 	(label "V4FREQ2"
-		(at 257.81 135.89 180)
+		(at 257.81 133.35 180)
 		(fields_autoplaced yes)
 		(effects
@@
 	)
 	(label "V1FREQ2"
-		(at 124.46 72.39 180)
-		(fields_autoplaced yes)
-		(effects
+		(at 124.46 69.85 180)
+		(fields_autoplaced yes)
+		(effects

Commit message: Updated sheet titles in modulation matrix and exported current rev1.0 schematic
Other:
- title: (none) -> Solstrejf Modulation Matrix Toplevel
Changed lines of the file:
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@@
 	(generator_version "8.0")
 	(paper "A4")
+	(title_block
+		(title "Solstrejf Modulation Matrix Toplevel")
+		(date "2024-08-24")
+		(rev "1.0")
+	)
 	(junction
 		(at 255.27 58.42)

Commit message: Updated voice board front-panel and mod-matrix
Created new dimensions to get a better physical layout of the 4x voice board control panels and the mod-matrix.
Exported .wrl 3D models of voice board front-panel and mod-matrix to create a MeshLab view.
Added MeshLab project files and new images aswell.
Parts:
- H1, H2, H3, H4: footprint MountingHole:MountingHole_3.2mm_M3 -> MountingHole:MountingHole_3.2mm_M3_DIN965
Changed lines of the file:
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@@
 			)
 		)
-		(property "Footprint" "MountingHole:MountingHole_3.2mm_M3"
+		(property "Footprint" "MountingHole:MountingHole_3.2mm_M3_DIN965"
 			(at 50.8 181.61 0)
 			(effects
@@
 			)
 		)
-		(property "Footprint" "MountingHole:MountingHole_3.2mm_M3"
+		(property "Footprint" "MountingHole:MountingHole_3.2mm_M3_DIN965"
 			(at 50.8 173.99 0)
 			(effects
@@
 			)
 		)
-		(property "Footprint" "MountingHole:MountingHole_3.2mm_M3"
+		(property "Footprint" "MountingHole:MountingHole_3.2mm_M3_DIN965"
 			(at 30.48 173.99 0)
 			(effects
@@
 			)
 		)
-		(property "Footprint" "MountingHole:MountingHole_3.2mm_M3"
+		(property "Footprint" "MountingHole:MountingHole_3.2mm_M3_DIN965"
 			(at 30.48 181.61 0)
 			(effects
