File: pcb/solstrejf-voiceboard-frontpanel/solstrejf-voiceboard-frontpanel.kicad_pcb (KiCad board)
At the start: 2 copper layers, 41.1 x 123.4 mm, 31 parts, among them J1 Conn_02x08_Odd_Even, J2 PIR Connector, J3 SJ335052B, SW1 TRIG, U1 TL972IP

Commit message: updated frontpanel resistor value and added 3D renders
Parts:
- R3: value 91k -> 56k

Commit message: updated frontpanel trig opamp output resistor due
- the weak pull-up on the ONESHOT env cause errors with creating zeros
Parts:
- R1: value 10k -> 1k
